File: kicad/ard-axlesim/ard-axlesim.kicad_pcb (KiCad board)
At the start: 2 copper layers, 68.6 x 53.3 mm, 27 parts, among them J1 Power, J10 SM04B-SRSS, J2 Digital/PWM, J3 Analog, J4 Digital/PWM, J5 Conn_01x03, J6 Conn_01x03, J7 Conn_01x03, J8 Conn_01x03, J9 SM04B-SRSS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

Commit message: Added DIP switch
Parts:
- added SW3: SW_DIP_x05, ISE_UltraLibrarian:CST_219SMT, F.Cu at (147.5, 63.4)
Routing:
- net /*5: track 0.00 -> 11.3 mm
- net /7: track 0.00 -> 11.3 mm
- net /4: track 0.00 -> 11.3 mm
- net /*6: track 0.00 -> 11.3 mm
- net /*3: track 0.00 -> 11.3 mm
- net GND: track 44.3 -> 54.5 mm, vias 7 -> 9

Commit message: Updates after review
Parts:
- added C3: 0.1uF, Capacitor_SMD:C_0805_2012Metric, F.Cu at (160.1, 89.0)
Connections:
- net +3V3 renamed ARD_3V3
- J1 pad 5: +5V -> ARD_5V
- J10 pad 2: +3.3V -> +5V
- J9 pad 2: +3.3V -> +5V
- R1 pad 2: +3.3V -> +5V
- R2 pad 2: +3.3V -> +5V
- R3 pad 2: +3.3V -> +5V
- R4 pad 2: +3.3V -> +5V
- SW2 pad 1: unconnected-(SW2-A-Pad1) -> Net-(SW2-A-Pad1)
- SW2 pad 4: unconnected-(SW2-A-Pad4) -> Net-(SW2-A-Pad1)
Routing:
- net +5V: track 0.00 -> 57.3 mm, vias 0 -> 4
- net +3.3V: track 57.3 -> 0.00 mm, vias 4 -> 0
- net GND: track 54.5 -> 44.7 mm, vias 9 -> 18
- net Net-(SW2-A-Pad1): track 0.00 -> 5.51 mm
- net /SCL/A5: track 36.7 -> 34.7 mm
- added copper zone on F.Cu, net /SCL/A5

Commit message: Added labels to DDIP switch
Other:
- board text added: "A B C D E"
Changed lines of the file:
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@@
-		(fp_text user "*"
-			(at -1.1176 -3.3636 0)
-			(layer "F.Fab")
-			(effects
-				(font
-					(size 1 1)
-					(thickness 0.15)
-				)
-			)
-		)
 		(fp_text user "*"
 			(at -1.1176 -3.3636 0)
 			(unlocked yes)
+			(layer "F.Fab")
+			(effects
+				(font
+					(size 1 1)
+					(thickness 0.15)
+				)
+			)
+		)
+		(fp_text user "*"
+			(at -1.1176 -3.3636 0)
 			(layer "F.Fab")
 			(effects
@@
 			)
 			(justify left bottom)
+		)
+	)
+	(gr_text "A  B  C  D  E"
+		(at 141.91 71.298 0)
+		(layer "F.SilkS")
+		(effects
+			(font
+				(size 1.524 1.016)
+				(thickness 0.1524)
+			)
+			(justify left bottom)
