File: kicad/ckt-axle-indicator/ckt-axle-indicator.kicad_pcb (KiCad board)
At the start: 2 copper layers, 50.8 x 25.4 mm, 9 parts, among them J1 SM04B-SRSS, J2 SM04B-SRSS, J3 SM04B-SRSS, J4 SM04B-SRSS

Commit message: Added text
Other:
- board text added: "CKT-AXLE-INDICATOR v1.0 ©2026 CC BY-SA"
Changed lines of the file:
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@@
+		)
+	)
+	(gr_text "CKT-AXLE-INDICATOR  v1.0\n©2026 CC BY-SA"
+		(at 152.4 122.428 0)
+		(layer "B.SilkS")
+		(effects
+			(font
+				(size 1.5 1.5)
+				(thickness 0.3)
+				(bold yes)
+			)
+			(justify bottom mirror)
 		)
 	)
