File: kicad/ckt-axle-bar/ckt-axle-bar-array.kicad_pcb (KiCad board)
At the start: 2 copper layers, 43.2 x 154.3 mm, 90 parts, among them J1 SM04B-SRSS, Q1 Q_Photo_NPN_EC, Q2 SSM6N357R

Commit message: Updated mousebites
Parts:
- removed KiKit_MB_1_5, KiKit_MB_2_5, KiKit_MB_3_5, KiKit_MB_4_5, KiKit_MB_5_5, KiKit_MB_6_5: NPTH, NPTH
- moved KiKit_MB_1_4 0.75 mm to (162.5, 44.4)
- moved KiKit_MB_2_4 0.75 mm to (134.5, 63.1)
- moved KiKit_MB_3_4 0.75 mm to (162.5, 87.8)
- moved KiKit_MB_4_4 0.75 mm to (134.5, 106.5)
- moved KiKit_MB_5_4 0.75 mm to (162.5, 131.2)
- moved KiKit_MB_6_4 0.75 mm to (134.5, 149.9)
- moved KiKit_MB_1_3 0.50 mm to (162.5, 43.4)
- moved KiKit_MB_2_3 0.50 mm to (134.5, 64.1)
- moved KiKit_MB_3_3 0.50 mm to (162.5, 86.8)
- moved KiKit_MB_4_3 0.50 mm to (134.5, 107.5)
- moved KiKit_MB_5_3 0.50 mm to (162.5, 130.2)
- moved KiKit_MB_6_3 0.50 mm to (134.5, 150.9)
- moved KiKit_MB_1_2 0.25 mm to (162.5, 42.4)
- moved KiKit_MB_2_2 0.25 mm to (134.5, 65.1)
- moved KiKit_MB_3_2 0.25 mm to (162.5, 85.8)
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